Commit message: Expand Humble tutorial examples and modularize sensors

File: ros2_ws/src/gazebo_tutorial_description/urdf/sensor_bot.urdf.xacro (robot description, xacro)
@@ -1,4 +1,13 @@
 <?xml version="1.0"?>
 <robot xmlns:xacro="http://www.ros.org/wiki/xacro" name="sensor_bot">
+  <!-- 센서 구현을 종류별 파일로 분리하고 여기서는 조합만 담당한다. -->
+  <xacro:include filename="$(find gazebo_tutorial_description)/urdf/sensors/sensor_common.xacro"/>
+  <xacro:include filename="$(find gazebo_tutorial_description)/urdf/sensors/imu_sensor.xacro"/>
+  <xacro:include filename="$(find gazebo_tutorial_description)/urdf/sensors/mono_rgb_camera.xacro"/>
+  <xacro:include filename="$(find gazebo_tutorial_description)/urdf/sensors/stereo_camera.xacro"/>
+  <xacro:include filename="$(find gazebo_tutorial_description)/urdf/sensors/rgbd_camera.xacro"/>
+  <xacro:include filename="$(find gazebo_tutorial_description)/urdf/sensors/fisheye_camera.xacro"/>
+  <xacro:include filename="$(find gazebo_tutorial_description)/urdf/sensors/lidar_2d.xacro"/>
+  <xacro:include filename="$(find gazebo_tutorial_description)/urdf/sensors/lidar_3d.xacro"/>
   <!--
     Gazebo Classic 11 + gazebo_ros_pkgs용 센서 실습 로봇.
@@ -38,29 +47,4 @@
         izz="${mass * (x * x + y * y) / 12.0}"/>
     </inertial>
-  </xacro:macro>
-  <xacro:macro name="sensor_box" params="name parent xyz size color:=sensor_gray">
-    <link name="${name}">
-      <visual>
-        <geometry>
-          <box size="${size}"/>
-        </geometry>
-        <material name="${color}"/>
-      </visual>
-      <xacro:box_inertial mass="0.05" x="0.04" y="0.04" z="0.04"/>
-    </link>
-    <joint name="${name}_joint" type="fixed">
-      <parent link="${parent}"/>
-      <child link="${name}"/>
-      <origin xyz="${xyz}" rpy="0 0 0"/>
-    </joint>
-  </xacro:macro>
-  <!-- ROS optical convention: +Z forward, +X right, +Y down. -->
-  <xacro:macro name="optical_frame" params="name parent">
-    <link name="${name}"/>
-    <joint name="${name}_joint" type="fixed">
-      <parent link="${parent}"/>
-      <child link="${name}"/>
-      <origin xyz="0 0 0" rpy="${-pi / 2.0} 0 ${-pi / 2.0}"/>
-    </joint>
   </xacro:macro>
   <!-- 바닥 투영 프레임. 차체 중심은 지면에서 0.18 m 위에 있다. -->
@@ -199,203 +183,31 @@
   </gazebo>
   <!-- IMU는 모든 프로필에서 사용한다. -->
-  <xacro:sensor_box name="imu_link" parent="base_link" xyz="0 0 0.10" size="0.05 0.04 0.02"/>
-  <gazebo reference="imu_link">
-    <sensor name="imu_sensor" type="imu">
-      <always_on>true</always_on>
-      <visualize>false</visualize>
-      <update_rate>100</update_rate>
-      <imu>
-        <angular_velocity>
-          <x><noise type="gaussian"><mean>0</mean><stddev>0.0002</stddev></noise></x>
-          <y><noise type="gaussian"><mean>0</mean><stddev>0.0002</stddev></noise></y>
-          <z><noise type="gaussian"><mean>0</mean><stddev>0.0002</stddev></noise></z>
-        </angular_velocity>
-        <linear_acceleration>
-          <x><noise type="gaussian"><mean>0</mean><stddev>0.017</stddev></noise></x>
-          <y><noise type="gaussian"><mean>0</mean><stddev>0.017</stddev></noise></y>
-          <z><noise type="gaussian"><mean>0</mean><stddev>0.017</stddev></noise></z>
-        </linear_acceleration>
-      </imu>
-      <plugin name="imu_ros" filename="libgazebo_ros_imu_sensor.so">
-        <ros>
-          <namespace>/</namespace>
-          <remapping>~/out:=imu/data</remapping>
-        </ros>
-        <frame_name>imu_link</frame_name>
-        <initial_orientation_as_reference>false</initial_orientation_as_reference>
-      </plugin>
-    </sensor>
-  </gazebo>
+  <xacro:gazebo_imu_sensor
+    prefix="imu" parent="base_link" xyz="0 0 0.10"
+    topic="imu/data" update_rate="100.0"
+    angular_stddev="0.0002" linear_stddev="0.017"/>
   <xacro:if value="${enable_cameras}">
-    <!-- 단안 카메라: L8 포맷이 sensor_msgs/Image의 mono8 encoding으로 변환된다. -->
-    <xacro:sensor_box name="camera_link" parent="base_link"
-      xyz="0.30 -0.12 0.07" size="0.06 0.05 0.05"/>
-    <xacro:optical_frame name="camera_optical_frame" parent="camera_link"/>
-    <gazebo reference="camera_link">
-      <sensor name="mono_camera_sensor" type="camera">
-        <always_on>true</always_on>
-        <visualize>true</visualize>
-        <update_rate>15</update_rate>
-        <camera name="mono">
-          <horizontal_fov>1.0471975512</horizontal_fov>
-          <image>
-            <width>320</width>
-            <height>240</height>
-            <format>L8</format>
-          </image>
-          <clip><near>0.05</near><far>30.0</far></clip>
-          <noise><type>gaussian</type><mean>0</mean><stddev>0.003</stddev></noise>
-        </camera>
-        <plugin name="mono_camera_ros" filename="libgazebo_ros_camera.so">
-          <ros><namespace>/</namespace></ros>
-          <camera_name>camera</camera_name>
-          <frame_name>camera_optical_frame</frame_name>
-        </plugin>
-      </sensor>
-    </gazebo>
-    <!-- 하나의 multicamera 센서가 같은 시각에 좌/우 영상을 렌더링한다. -->
-    <xacro:sensor_box name="stereo_camera_link" parent="base_link"
-      xyz="0.30 0 0.15" size="0.06 0.12 0.04"/>
-    <xacro:optical_frame name="stereo_camera_optical_frame" parent="stereo_camera_link"/>
-    <gazebo reference="stereo_camera_link">
-      <sensor name="stereo_camera_sensor" type="multicamera">
-        <always_on>true</always_on>
-        <visualize>false</visualize>
-        <update_rate>10</update_rate>
-        <camera name="left">
-          <pose>0 0.04 0 0 0 0</pose>
-          <horizontal_fov>1.0471975512</horizontal_fov>
-          <image><width>320</width><height>240</height><format>R8G8B8</format></image>
-          <clip><near>0.05</near><far>30.0</far></clip>
-          <noise><type>gaussian</type><mean>0</mean><stddev>0.003</stddev></noise>
-        </camera>
-        <camera name="right">
-          <pose>0 -0.04 0 0 0 0</pose>
-          <horizontal_fov>1.0471975512</horizontal_fov>
-          <image><width>320</width><height>240</height><format>R8G8B8</format></image>
-          <clip><near>0.05</near><far>30.0</far></clip>
-          <noise><type>gaussian</type><mean>0</mean><stddev>0.003</stddev></noise>
-        </camera>
-        <plugin name="stereo_camera_ros" filename="libgazebo_ros_camera.so">
-          <ros><namespace>/</namespace></ros>
-          <camera_name>stereo</camera_name>
-          <frame_name>stereo_camera_optical_frame</frame_name>
-          <hack_baseline>0.08</hack_baseline>
-        </plugin>
-      </sensor>
-    </gazebo>
-    <!-- depth 센서는 RGB, depth, CameraInfo, PointCloud2를 한 플러그인에서 발행한다. -->
-    <xacro:sensor_box name="rgbd_camera_link" parent="base_link"
-      xyz="0.30 0.12 0.07" size="0.06 0.07 0.05" color="sensor_green"/>
-    <xacro:optical_frame name="rgbd_camera_optical_frame" parent="rgbd_camera_link"/>
-    <gazebo reference="rgbd_camera_link">
-      <sensor name="rgbd_camera_sensor" type="depth">
-        <always_on>true</always_on>
-        <visualize>false</visualize>
-        <update_rate>10</update_rate>
-        <camera name="rgbd">
-          <horizontal_fov>1.0471975512</horizontal_fov>
-          <image><width>320</width><height>240</height><format>R8G8B8</format></image>
-          <clip><near>0.10</near><far>12.0</far></clip>
-          <noise><type>gaussian</type><mean>0</mean><stddev>0.002</stddev></noise>
-        </camera>
-        <plugin name="rgbd_camera_ros" filename="libgazebo_ros_camera.so">
-          <ros><namespace>/</namespace></ros>
-          <camera_name>rgbd</camera_name>
-          <frame_name>rgbd_camera_optical_frame</frame_name>
-          <min_depth>0.10</min_depth>
-          <max_depth>12.0</max_depth>
-        </plugin>
-      </sensor>
-    </gazebo>
-    <!-- Gazebo 11 wide-angle camera의 equidistant 렌즈 모델. -->
-    <xacro:sensor_box name="fisheye_camera_link" parent="base_link"
-      xyz="0.06 -0.10 0.22" size="0.06 0.06 0.05" color="sensor_green"/>
-    <xacro:optical_frame name="fisheye_camera_optical_frame" parent="fisheye_camera_link"/>
-    <gazebo reference="fisheye_camera_link">
-      <sensor name="fisheye_camera_sensor" type="wideanglecamera">
-        <always_on>true</always_on>
-        <visualize>true</visualize>
-        <update_rate>10</update_rate>
-        <camera name="fisheye">
-          <horizontal_fov>3.1415926535</horizontal_fov>
-          <image><width>320</width><height>240</height><format>R8G8B8</format></image>
-          <clip><near>0.05</near><far>30.0</far></clip>
-          <lens>
-            <type>equidistant</type>
-            <scale_to_hfov>true</scale_to_hfov>
-            <cutoff_angle>1.5707</cutoff_angle>
-            <env_texture_size>512</env_texture_size>
-          </lens>
-        </camera>
-        <plugin name="fisheye_camera_ros" filename="libgazebo_ros_camera.so">
-          <ros><namespace>/</namespace></ros>
-          <camera_name>fisheye</camera_name>
-          <frame_name>fisheye_camera_optical_frame</frame_name>
-        </plugin>
-      </sensor>
-    </gazebo>
+    <xacro:gazebo_mono_rgb_camera
+      prefix="camera" parent="base_link" xyz="0.30 -0.12 0.07"
+      camera_name="camera" format="L8" update_rate="15.0"/>
+    <xacro:gazebo_stereo_camera
+      prefix="stereo_camera" parent="base_link" xyz="0.30 0 0.15"
+      camera_name="stereo" baseline="0.08" update_rate="10.0"/>
+    <xacro:gazebo_rgbd_camera
+      prefix="rgbd_camera" parent="base_link" xyz="0.30 0.12 0.07"
+      camera_name="rgbd" min_depth="0.10" max_depth="12.0" update_rate="10.0"/>
+    <xacro:gazebo_fisheye_camera
+      prefix="fisheye_camera" parent="base_link" xyz="0.06 -0.10 0.22"
+      camera_name="fisheye" horizontal_fov="3.1415926535"
+      lens_type="equidistant" env_texture_size="512" update_rate="10.0"/>
   </xacro:if>
   <xacro:if value="${enable_lidars}">
-    <!-- 수평 한 줄만 스캔하므로 LaserScan으로 내보낸다. -->
-    <xacro:sensor_box name="lidar_2d_link" parent="base_link"
-      xyz="0.13 0 0.22" size="0.07 0.07 0.05"/>
-    <gazebo reference="lidar_2d_link">
-      <sensor name="lidar_2d_sensor" type="ray">
-        <always_on>true</always_on>
-        <visualize>true</visualize>
-        <update_rate>15</update_rate>
-        <ray>
-          <scan>
-            <horizontal>
-              <samples>720</samples><resolution>1</resolution>
-              <min_angle>-${pi}</min_angle><max_angle>${pi}</max_angle>
-            </horizontal>
-          </scan>
-          <range><min>0.12</min><max>15.0</max><resolution>0.01</resolution></range>
-          <noise><type>gaussian</type><mean>0</mean><stddev>0.01</stddev></noise>
-        </ray>
-        <plugin name="lidar_2d_ros" filename="libgazebo_ros_ray_sensor.so">
-          <ros>
-            <namespace>/</namespace>
-            <remapping>~/out:=scan</remapping>
-          </ros>
-          <output_type>sensor_msgs/LaserScan</output_type>
-          <frame_name>lidar_2d_link</frame_name>
-        </plugin>
-      </sensor>
-    </gazebo>
-    <!-- 수직 채널을 가진 ray 센서는 PointCloud2로 내보낸다. -->
-    <xacro:sensor_box name="lidar_3d_link" parent="base_link"
-      xyz="-0.12 0 0.22" size="0.09 0.09 0.07" color="sensor_green"/>
-    <gazebo reference="lidar_3d_link">
-      <sensor name="lidar_3d_sensor" type="ray">
-        <always_on>true</always_on>
-        <visualize>false</visualize>
-        <update_rate>10</update_rate>
-        <ray>
-          <scan>
-            <horizontal>
-              <samples>360</samples><resolution>1</resolution>
-              <min_angle>-${pi}</min_angle><max_angle>${pi}</max_angle>
-            </horizontal>
-            <vertical>
-              <samples>16</samples><resolution>1</resolution>
-              <min_angle>-0.261799</min_angle><max_angle>0.261799</max_angle>
-            </vertical>
-          </scan>
-          <range><min>0.20</min><max>20.0</max><resolution>0.02</resolution></range>
-          <noise><type>gaussian</type><mean>0</mean><stddev>0.015</stddev></noise>
-        </ray>
-        <plugin name="lidar_3d_ros" filename="libgazebo_ros_ray_sensor.so">
-          <ros>
-            <namespace>/</namespace>
-            <remapping>~/out:=points</remapping>
-          </ros>
-          <output_type>sensor_msgs/PointCloud2</output_type>
-          <frame_name>lidar_3d_link</frame_name>
-        </plugin>
-      </sensor>
-    </gazebo>
+    <xacro:gazebo_lidar_2d
+      prefix="lidar_2d" parent="base_link" xyz="0.13 0 0.22"
+      topic="scan" samples="720" update_rate="15.0"/>
+    <xacro:gazebo_lidar_3d
+      prefix="lidar_3d" parent="base_link" xyz="-0.12 0 0.22"
+      topic="points" horizontal_samples="360" vertical_samples="16"
+      update_rate="10.0"/>
   </xacro:if>
 </robot>

Commit message: 센서 로봇의 전방 전도 방지

File: ros2_ws/src/gazebo_tutorial_description/urdf/sensor_bot.urdf.xacro (robot description, xacro)
@@ -27,4 +27,8 @@
   <xacro:property name="wheel_width" value="0.045"/>
   <xacro:property name="wheel_separation" value="0.43"/>
+  <!-- all 프로필의 전방 센서 모멘트를 상쇄하는 후방 caster 겸 counterweight. -->
+  <xacro:property name="caster_radius" value="0.05"/>
+  <xacro:property name="caster_mass" value="1.20"/>
+  <xacro:property name="caster_x" value="-0.20"/>
   <material name="body_blue">
     <color rgba="0.10 0.35 0.75 1.0"/>
@@ -117,5 +121,5 @@
     <visual>
       <geometry>
-        <sphere radius="0.05"/>
+        <sphere radius="${caster_radius}"/>
       </geometry>
       <material name="dark_gray"/>
@@ -123,10 +127,15 @@
     <collision>
       <geometry>
-        <sphere radius="0.05"/>
+        <sphere radius="${caster_radius}"/>
       </geometry>
     </collision>
     <inertial>
-      <mass value="0.20"/>
-      <inertia ixx="0.0002" ixy="0" ixz="0" iyy="0.0002" iyz="0" izz="0.0002"/>
+      <mass value="${caster_mass}"/>
+      <inertia
+        ixx="${2.0 * caster_mass * caster_radius * caster_radius / 5.0}"
+        ixy="0" ixz="0"
+        iyy="${2.0 * caster_mass * caster_radius * caster_radius / 5.0}"
+        iyz="0"
+        izz="${2.0 * caster_mass * caster_radius * caster_radius / 5.0}"/>
     </inertial>
   </link>
@@ -134,5 +143,5 @@
     <parent link="base_link"/>
     <child link="caster_link"/>
-    <origin xyz="-0.20 0 -0.13" rpy="0 0 0"/>
+    <origin xyz="${caster_x} 0 -0.13" rpy="0 0 0"/>
   </joint>
   <gazebo reference="caster_link">
