Commit message: Humble: revise Korean tutorials and correct Classic sensors, TF, and vehicle motion

File: ros2_ws/src/f1_robot_model/urdf/3dlidar.xacro (robot description, xacro)
@@ -3,8 +3,8 @@
     <joint name="lidar_base_joint" type="fixed">
         <parent link="base_link"/>
-        <child link="base"/>
-        <origin xyz="0.2 0 0.1" rpy="0 0 0"/>
+        <child link="lidar_3d_base"/>
+        <origin xyz="0 0 0.18" rpy="0 0 0"/>
     </joint>
-    <link name="base">
+    <link name="lidar_3d_base">
         <visual>
             <geometry>
@@ -22,13 +22,13 @@
         </xacro:inertial_cylinder-->
     </link>
-    <gazebo reference="base">
+    <gazebo reference="lidar_3d_base">
         <material>Gazebo/Red</material>
     </gazebo>
     <joint name="laser_joint" type="fixed">
-        <parent link="base"/>
-        <child link="top"/>
+        <parent link="lidar_3d_base"/>
+        <child link="lidar_3d_link"/>
         <origin xyz="0 0 0.067" rpy="0 0 0"/>
     </joint>
-    <link name="top">
+    <link name="lidar_3d_link">
         <visual>
             <geometry>
@@ -46,5 +46,5 @@
         </xacro:inertial_cylinder-->
     </link>
-    <gazebo reference="top">
+    <gazebo reference="lidar_3d_link">
         <material>Gazebo/Red</material>
         <sensor type="ray" name="velodyne2-HDL32E">
@@ -80,10 +80,10 @@
             <plugin name="gazebo_ros_laser_controller" filename="libgazebo_ros_velodyne_laser.so">
                 <ros>
-                    <namespace>/velodyne2</namespace>
-                    <remapping>~/out:=velodyne_points2</remapping>
+                    <namespace>/lidar_3d</namespace>
+                    <remapping>~/out:=points</remapping>
                 </ros>
-                <frame_name>top</frame_name>
+                <frame_name>lidar_3d_link</frame_name>
                 <organize_cloud>false</organize_cloud>
-                <min_range>0.9</min_range>
+                <min_range>0.3</min_range>
                 <max_range>130.0</max_range>
                 <gaussian_noise>0.008</gaussian_noise>

File: ros2_ws/src/f1_robot_model/urdf/depth_camera.xacro (robot description, xacro)
@@ -22,7 +22,7 @@
     <gazebo reference="camera_link">
         <material>Gazebo/Blue</material>
-        <sensor name="camera" type="depth">
+        <sensor name="depth_camera_sensor" type="depth">
             <pose> 0 0 0 0 0 0 </pose>
-            <visualize>true</visualize>
+            <visualize>false</visualize>
             <update_rate>30</update_rate>
             <camera>
@@ -30,6 +30,6 @@
                 <image>
                     <format>B8G8R8</format>
-                    <width>640</width>
-                    <height>480</height>
+                    <width>320</width>
+                    <height>240</height>
                 </image>
                 <clip>
@@ -44,8 +44,10 @@
             </camera>
             <plugin name="camera_controller" filename="libgazebo_ros_camera.so">
+                <camera_name>camera</camera_name>
+                <cx>159.5</cx>
+                <cy>119.5</cy>
                 <frame_name>camera_link_optical</frame_name>
                 <min_depth>0.05</min_depth>
                 <max_depth>8.0</max_depth>
-                <updateRate>30.0</updateRate>
             </plugin>
         </sensor>

File: ros2_ws/src/f1_robot_model/urdf/gps.xacro (robot description, xacro)
@@ -11,4 +11,5 @@
                     <remapping>~/out:=data</remapping>
                 </ros>
+                <frame_name>gps</frame_name>
             </plugin>
         </sensor>

File: ros2_ws/src/f1_robot_model/urdf/imu.xacro (robot description, xacro)
@@ -55,5 +55,6 @@
                     <remapping>~/out:=data</remapping>
                 </ros>
-                <initialOrientationAsReference>true</initialOrientationAsReference>
+                <frame_name>imu</frame_name>
+                <initial_orientation_as_reference>false</initial_orientation_as_reference>
             </plugin>
         </sensor>

File: ros2_ws/src/f1_robot_model/urdf/left_camera.xacro (robot description, xacro)
@@ -24,7 +24,7 @@
     <gazebo reference="left_camera_link">
         <material>Gazebo/Blue</material>
-        <sensor name="camera" type="camera">
+        <sensor name="left_camera_sensor" type="camera">
             <pose> 0 0 0 0 0 0 </pose>
-            <visualize>true</visualize>
+            <visualize>false</visualize>
             <update_rate>30</update_rate>
             <camera>
@@ -32,6 +32,6 @@
                 <image>
                     <format>B8G8R8</format>
-                    <width>640</width>
-                    <height>480</height>
+                    <width>320</width>
+                    <height>240</height>
                 </image>
                 <distortion>
@@ -50,11 +50,8 @@
             </camera>
             <plugin name="left_camera_controller" filename="libgazebo_ros_camera.so">
-                <ros>
-                    <namespace>left_camera</namespace>
-                    <remapping>camera_info:=left_camera/camera_info</remapping>
-                    <remapping>image_raw:=left_camera/image_raw</remapping>
-                </ros>
+                <camera_name>left_camera</camera_name>
+                <cx>159.5</cx>
+                <cy>119.5</cy>
                 <frame_name>left_camera_link_optical</frame_name>
-                <updateRate>30.0</updateRate>
             </plugin>
         </sensor>

File: ros2_ws/src/f1_robot_model/urdf/macros.xacro (robot description, xacro)
@@ -42,5 +42,5 @@
   <geometry>
     <!-- <mesh filename="package://f1_robot_model/meshes/chassis.STL" /> -->
-    <mesh filename="file://$(find f1_robot_model)/meshes/chassis.STL"/>
+    <mesh filename="package://f1_robot_model/meshes/chassis.STL"/>
   </geometry>
 </xacro:macro>
@@ -49,5 +49,5 @@
   <geometry>
     <!-- <mesh filename="package://f1_robot_model/meshes/left_rear_wheel.STL" /> -->
-    <mesh filename="file://$(find f1_robot_model)/meshes/left_rear_wheel.STL"/>
+    <mesh filename="package://f1_robot_model/meshes/left_rear_wheel.STL"/>
   </geometry>
 </xacro:macro>
@@ -56,5 +56,5 @@
   <geometry>
     <!-- <mesh filename="package://f1_robot_model/meshes/right_rear_wheel.STL" /> -->
-    <mesh filename="file://$(find f1_robot_model)/meshes/right_rear_wheel.STL"/>
+    <mesh filename="package://f1_robot_model/meshes/right_rear_wheel.STL"/>
   </geometry>
 </xacro:macro>
@@ -63,5 +63,5 @@
   <geometry>
     <!-- <mesh filename="package://f1_robot_model/meshes/left_front_wheel.STL" /> -->
-    <mesh filename="file://$(find f1_robot_model)/meshes/left_front_wheel.STL"/>
+    <mesh filename="package://f1_robot_model/meshes/left_front_wheel.STL"/>
   </geometry>
 </xacro:macro>
@@ -70,5 +70,5 @@
   <geometry>
     <!-- <mesh filename="package://f1_robot_model/meshes/right_front_wheel.STL" /> -->
-    <mesh filename="file://$(find f1_robot_model)/meshes/right_front_wheel.STL"/>
+    <mesh filename="package://f1_robot_model/meshes/right_front_wheel.STL"/>
   </geometry>
 </xacro:macro>
@@ -77,5 +77,5 @@
   <geometry>
     <!-- <mesh filename="package://f1_robot_model/meshes/left_steering_hinge.STL" /> -->
-    <mesh filename="file://$(find f1_robot_model)/meshes/left_steering_hinge.STL"/>
+    <mesh filename="package://f1_robot_model/meshes/left_steering_hinge.STL"/>
   </geometry>
 </xacro:macro>
@@ -84,5 +84,5 @@
   <geometry>
     <!-- <mesh filename="package://f1_robot_model/meshes/right_steering_hinge.STL" /> -->
-    <mesh filename="file://$(find f1_robot_model)/meshes/right_steering_hinge.STL"/>
+    <mesh filename="package://f1_robot_model/meshes/right_steering_hinge.STL"/>
   </geometry>
 </xacro:macro>

File: ros2_ws/src/f1_robot_model/urdf/racecar.urdf (robot description, URDF)
Before this commit: robot racecar, 12 links, 11 joints
Links:
- link chassis: geometry collision box size=0.36 0.18 0.035
- link laser: geometry collision box size=0.1 0.1 0.1; visual mesh filename=package://f1_robot_model/meshes/hokuyo.dae
Joints:
- joint right_steering_hinge_joint: type continuous -> revolute

File: ros2_ws/src/f1_robot_model/urdf/right_camera.xacro (robot description, xacro)
@@ -24,7 +24,7 @@
     <gazebo reference="right_camera_link">
         <material>Gazebo/Blue</material>
-        <sensor name="camera" type="camera">
+        <sensor name="right_camera_sensor" type="camera">
             <pose>0 0 0 0 0 0</pose>
-            <visualize>true</visualize>
+            <visualize>false</visualize>
             <update_rate>30</update_rate>
             <camera>
@@ -32,6 +32,6 @@
                 <image>
                     <format>B8G8R8</format>
-                    <width>640</width>
-                    <height>480</height>
+                    <width>320</width>
+                    <height>240</height>
                 </image>
                 <distortion>
@@ -50,11 +50,9 @@
             </camera>
             <plugin name="right_camera_controller" filename="libgazebo_ros_camera.so">
-                <ros>
-                    <namespace>right_camera</namespace>
-                    <remapping>camera_info:=right_camera/camera_info</remapping>
-                    <remapping>image_raw:=right_camera/image_raw</remapping>
-                </ros>
+                <camera_name>right_camera</camera_name>
+                <hack_baseline>0.2</hack_baseline>
+                <cx>159.5</cx>
+                <cy>119.5</cy>
                 <frame_name>right_camera_link_optical</frame_name>
-                <updateRate>30.0</updateRate>
             </plugin>
         </sensor>

File: ros2_ws/src/gazebo_tutorial_description/urdf/sensors/mono_rgb_camera.xacro (robot description, xacro)
@@ -29,4 +29,7 @@
           <camera_name>${camera_name}</camera_name>
           <frame_name>${prefix}_optical_frame</frame_name>
+          <!-- 픽셀 인덱스 0..width-1, 0..height-1의 중앙을 사용한다. -->
+          <cx>${(width - 1) / 2.0}</cx>
+          <cy>${(height - 1) / 2.0}</cy>
         </plugin>
       </sensor>

File: ros2_ws/src/gazebo_tutorial_description/urdf/sensors/rgbd_camera.xacro (robot description, xacro)
@@ -25,4 +25,7 @@
           <camera_name>${camera_name}</camera_name>
           <frame_name>${prefix}_optical_frame</frame_name>
+          <!-- gazebo_ros_camera의 점군 생성식과 CameraInfo의 광학 중심을 맞춘다. -->
+          <cx>${(width - 1) / 2.0}</cx>
+          <cy>${(height - 1) / 2.0}</cy>
           <min_depth>${min_depth}</min_depth>
           <max_depth>${max_depth}</max_depth>

File: ros2_ws/src/gazebo_tutorial_description/urdf/sensors/sensor_common.xacro (robot description, xacro)
@@ -32,10 +32,10 @@
   </xacro:macro>
   <!-- REP-103 optical frame은 +Z 전방, +X 오른쪽, +Y 아래쪽을 사용한다. -->
-  <xacro:macro name="sensor_optical_frame" params="frame_name parent">
+  <xacro:macro name="sensor_optical_frame" params="frame_name parent xyz:='0 0 0'">
     <link name="${frame_name}"/>
     <joint name="${frame_name}_joint" type="fixed">
       <parent link="${parent}"/>
       <child link="${frame_name}"/>
-      <origin xyz="0 0 0" rpy="${-pi / 2.0} 0 ${-pi / 2.0}"/>
+      <origin xyz="${xyz}" rpy="${-pi / 2.0} 0 ${-pi / 2.0}"/>
     </joint>
   </xacro:macro>

File: ros2_ws/src/gazebo_tutorial_description/urdf/sensors/stereo_camera.xacro (robot description, xacro)
@@ -8,12 +8,20 @@
       link_name="${prefix}_link" parent="${parent}" xyz="${xyz}" rpy="${rpy}"
       size_x="0.06" size_y="0.12" size_z="0.04" color="sensor_gray"/>
-    <xacro:sensor_optical_frame frame_name="${prefix}_optical_frame" parent="${prefix}_link"/>
+    <!-- 두 광학 프레임의 위치를 실제 렌즈 중심과 맞춘다. +Y가 로봇의 왼쪽이다. -->
+    <xacro:sensor_optical_frame
+      frame_name="${prefix}_left_optical_frame" parent="${prefix}_link"
+      xyz="0 ${baseline / 2.0} 0"/>
+    <xacro:sensor_optical_frame
+      frame_name="${prefix}_right_optical_frame" parent="${prefix}_link"
+      xyz="0 ${-baseline / 2.0} 0"/>
+    <!-- Classic multicamera 플러그인은 frame_name과 투영행렬 설정을 공유한다.
+         좌우 위치와 오른쪽 P[3]를 정확하게 표현하기 위해 센서를 둘로 나눈다. -->
     <gazebo reference="${prefix}_link">
-      <sensor name="${prefix}_sensor" type="multicamera">
+      <sensor name="${prefix}_left_sensor" type="camera">
+        <pose>0 ${baseline / 2.0} 0 0 0 0</pose>
         <always_on>true</always_on>
         <visualize>${visualize}</visualize>
         <update_rate>${update_rate}</update_rate>
         <camera name="left">
-          <pose>0 ${baseline / 2.0} 0 0 0 0</pose>
           <horizontal_fov>${horizontal_fov}</horizontal_fov>
           <image><width>${width}</width><height>${height}</height><format>R8G8B8</format></image>
@@ -21,6 +29,19 @@
           <noise><type>gaussian</type><mean>0</mean><stddev>${image_noise_stddev}</stddev></noise>
         </camera>
+        <plugin name="${prefix}_left_ros" filename="libgazebo_ros_camera.so">
+          <ros><namespace>${ros_namespace}</namespace></ros>
+          <camera_name>${camera_name}/left</camera_name>
+          <frame_name>${prefix}_left_optical_frame</frame_name>
+          <cx>${(width - 1) / 2.0}</cx>
+          <cy>${(height - 1) / 2.0}</cy>
+          <hack_baseline>0.0</hack_baseline>
+        </plugin>
+      </sensor>
+      <sensor name="${prefix}_right_sensor" type="camera">
+        <pose>0 ${-baseline / 2.0} 0 0 0 0</pose>
+        <always_on>true</always_on>
+        <visualize>${visualize}</visualize>
+        <update_rate>${update_rate}</update_rate>
         <camera name="right">
-          <pose>0 ${-baseline / 2.0} 0 0 0 0</pose>
           <horizontal_fov>${horizontal_fov}</horizontal_fov>
           <image><width>${width}</width><height>${height}</height><format>R8G8B8</format></image>
@@ -28,8 +49,12 @@
           <noise><type>gaussian</type><mean>0</mean><stddev>${image_noise_stddev}</stddev></noise>
         </camera>
-        <plugin name="${prefix}_ros" filename="libgazebo_ros_camera.so">
+        <plugin name="${prefix}_right_ros" filename="libgazebo_ros_camera.so">
           <ros><namespace>${ros_namespace}</namespace></ros>
-          <camera_name>${camera_name}</camera_name>
-          <frame_name>${prefix}_optical_frame</frame_name>
+          <camera_name>${camera_name}/right</camera_name>
+          <frame_name>${prefix}_right_optical_frame</frame_name>
+          <cx>${(width - 1) / 2.0}</cx>
+          <cy>${(height - 1) / 2.0}</cy>
+          <!-- CameraInfo 오른쪽 투영행렬: P[3] = -fx * baseline [pixel*m]. -->
+          <hack_baseline>${baseline}</hack_baseline>
         </plugin>
       </sensor>
